File: SerialOLED.sch (EAGLE design)
At the start: 23 parts, among them IC3 MCP1703CB, U1 ATMEGA328, X1 16 MHz

Commit message: Solder-bridge for FTDI reset replaced with a capacitor
Parts:
- removed JP4: (no value), SparkFun:JUMPER-2SMD-NO
- added C6: 0.1u, SparkFun:CAP0603-CAP
Connections:
- net DTR: now also C6.2; no longer JP4.2
- net RST: now also C6.1; no longer JP4.1
Other:
- moved on the sheet: R1, RST
Changed lines of the file:
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@@
 <setting verticaltext="up"/>
 </settings>
-<grid distance="0.1" unitdist="inch" unit="inch" style="lines" multiple="1" display="no" altdistance="0.01" altunitdist="inch" altunit="inch"/>
+<grid distance="25" unitdist="mil" unit="mil" style="lines" multiple="1" display="no" altdistance="5" altunitdist="mil" altunit="mil"/>
 <layers>
 <layer number="1" name="Top" color="4" fill="1" visible="no" active="no"/>
@@
 <part name="JP2" library="SparkFun" deviceset="M06" device="SIP_LOCK" value="HOST"/>
 <part name="JP3" library="SparkFun" deviceset="M06" device="SIP_LOCK" value="DEVICE"/>
-<part name="JP4" library="SparkFun" deviceset="JUMPER-2" device="SMD-NO"/>
+<part name="C6" library="SparkFun" deviceset="CAP" device="0603-CAP" value="0.1u"/>
 </parts>
 <sheets>
@@
 </plain>
 <instances>
-<instance part="R1" gate="G$1" x="48.895" y="162.56" rot="R180"/>
+<instance part="R1" gate="G$1" x="48.895" y="166.37" rot="R180"/>
 <instance part="C2" gate="G$1" x="195.58" y="68.58"/>
 <instance part="SUPPLY3" gate="1" x="157.48" y="81.28"/>
@@
 <instance part="SUPPLY2" gate="GND" x="41.91" y="131.445" rot="R270"/>
 <instance part="U$6" gate="G$1" x="58.42" y="71.12"/>
-<instance part="RST" gate="G$1" x="47.625" y="154.94" smashed="yes">
-<attribute name="NAME" x="45.085" y="156.972" size="1.27" layer="95" font="vector"/>
+<instance part="RST" gate="G$1" x="47.625" y="160.655" smashed="yes">
+<attribute name="NAME" x="45.085" y="162.687" size="1.27" layer="95" font="vector"/>
 </instance>
 <instance part="PB2" gate="G$1" x="139.7" y="129.54" rot="R270"/>
@@
 <instance part="SUPPLY1" gate="GND" x="132.08" y="93.98"/>
 <instance part="SUPPLY4" gate="1" x="132.08" y="137.16"/>
-<instance part="3.3V" gate="1" x="43.18" y="162.56" rot="R90"/>
+<instance part="3.3V" gate="1" x="43.18" y="166.37" rot="R90"/>
 <instance part="SUPPLY6" gate="1" x="43.18" y="142.24" rot="R90"/>
-<instance part="SUPPLY5" gate="GND" x="41.91" y="154.94" rot="R270"/>
+<instance part="SUPPLY5" gate="GND" x="41.91" y="160.655" rot="R270"/>
 <instance part="SJ1" gate="G$1" x="172.72" y="144.78" rot="R180"/>
 <instance part="SJ2" gate="G$1" x="162.56" y="137.16" rot="R180"/>
@@
 <instance part="JP2" gate="G$1" x="93.98" y="68.58"/>
 <instance part="JP3" gate="G$1" x="129.54" y="68.58"/>
-<instance part="JP4" gate="A" x="162.56" y="104.14" rot="R90"/>
+<instance part="C6" gate="G$1" x="46.355" y="154.94" rot="MR90"/>
 </instances>
 <busses>
@@
 <segment>
 <pinref part="RST" gate="G$1" pin="1"/>
-<wire x1="45.085" y1="154.94" x2="44.45" y2="154.94" width="0.1524" layer="91"/>
+<wire x1="45.085" y1="160.655" x2="44.45" y2="160.655" width="0.1524" layer="91"/>
 <pinref part="SUPPLY5" gate="GND" pin="GND"/>
 </segment>
@@
 <pinref part="R1" gate="G$1" pin="1"/>
 <pinref part="U1" gate="G$1" pin="PC6(/RESET)"/>
-<wire x1="53.975" y1="162.56" x2="54.61" y2="162.56" width="0.1524" layer="91"/>
-<wire x1="54.61" y1="162.56" x2="54.61" y2="154.94" width="0.1524" layer="91"/>
+<wire x1="53.975" y1="166.37" x2="54.61" y2="166.37" width="0.1524" layer="91"/>
+<wire x1="54.61" y1="166.37" x2="54.61" y2="160.655" width="0.1524" layer="91"/>
+<wire x1="54.61" y1="160.655" x2="54.61" y2="154.94" width="0.1524" layer="91"/>
 <wire x1="54.61" y1="154.94" x2="54.61" y2="149.86" width="0.1524" layer="91"/>
 <wire x1="54.61" y1="149.86" x2="55.88" y2="149.86" width="0.1524" layer="91"/>
 <wire x1="54.61" y1="149.86" x2="40.64" y2="149.86" width="0.1524" layer="91"/>
 <junction x="54.61" y="149.86"/>
-<label x="43.18" y="147.32" size="1.778" layer="95"/>
+<label x="40.64" y="149.86" size="1.778" layer="95"/>
 <pinref part="RST" gate="G$1" pin="2"/>
-<wire x1="54.61" y1="154.94" x2="50.165" y2="154.94" width="0.1524" layer="91"/>
+<wire x1="54.61" y1="160.655" x2="50.165" y2="160.655" width="0.1524" layer="91"/>
+<junction x="54.61" y="160.655"/>
+<wire x1="51.435" y1="154.94" x2="54.61" y2="154.94" width="0.1524" layer="91"/>
 <junction x="54.61" y="154.94"/>
+<pinref part="C6" gate="G$1" pin="1"/>
 </segment>
 <segment>
 <pinref part="U$6" gate="G$1" pin="P$3"/>
 <wire x1="48.26" y1="66.04" x2="40.64" y2="66.04" width="0.1524" layer="91"/>
-</segment>
-<segment>
-<pinref part="JP4" gate="A" pin="1"/>
-<wire x1="165.1" y1="104.14" x2="172.72" y2="104.14" width="0.1524" layer="91"/>
-<label x="167.64" y="104.14" size="1.778" layer="95"/>
 </segment>
 </net>
@@
 <pinref part="3.3V" gate="1" pin="VCC"/>
 <pinref part="R1" gate="G$1" pin="2"/>
-<wire x1="43.18" y1="162.56" x2="43.815" y2="162.56" width="0.1524" layer="91"/>
+<wire x1="43.18" y1="166.37" x2="43.815" y2="166.37" width="0.1524" layer="91"/>
 </segment>
 <segment>
@@
 </segment>
 <segment>
-<pinref part="JP4" gate="A" pin="2"/>
-<wire x1="165.1" y1="106.68" x2="172.72" y2="106.68" width="0.1524" layer="91"/>
-<label x="167.64" y="106.68" size="1.778" layer="95"/>
-</segment>
-</net>
+<pinref part="C6" gate="G$1" pin="2"/>
+<wire x1="43.815" y1="154.94" x2="40.64" y2="154.94" width="0.1524" layer="91"/>
+<label x="40.64" y="154.94" size="1.778" layer="95"/>
+</segment>
+</net>
