File: SerialOLED.sch (EAGLE design)
At the start: 23 parts, among them IC3 MCP1703CB, U1 ATMEGA328, X1 16 MHz

Commit message: Board fixes and new pictures
Connections:
- net RXD: now also JP3.5; no longer JP3.4
- net TXD: now also JP3.4; no longer JP3.5
Changed lines of the file:
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@@
 </segment>
 <segment>
-<wire x1="134.62" y1="73.66" x2="144.78" y2="73.66" width="0.1524" layer="91"/>
-<label x="137.16" y="73.66" size="1.778" layer="95"/>
-<pinref part="JP3" gate="G$1" pin="5"/>
+<pinref part="JP3" gate="G$1" pin="4"/>
+<wire x1="134.62" y1="71.12" x2="144.78" y2="71.12" width="0.1524" layer="91"/>
+<label x="137.16" y="71.12" size="1.778" layer="95"/>
 </segment>
 </net>
@@
 </segment>
 <segment>
-<wire x1="134.62" y1="71.12" x2="144.78" y2="71.12" width="0.1524" layer="91"/>
-<label x="137.16" y="71.12" size="1.778" layer="95"/>
-<pinref part="JP3" gate="G$1" pin="4"/>
+<pinref part="JP3" gate="G$1" pin="5"/>
+<wire x1="134.62" y1="73.66" x2="144.78" y2="73.66" width="0.1524" layer="91"/>
+<label x="137.16" y="73.66" size="1.778" layer="95"/>
 </segment>
 </net>
